File: hardwareDesign/shield/adc.kicad_sch (KiCad schematic)
At the start: 1 part, among them U1 MCP3208

Commit message: Finished schematic and PCB for jetson Nano Sheild
Parts:
- added C17: 10uf_0603_25V, capacitors:SMD_0603[1608], symbol capacitors_smd:10uf_0603_25V
- added C18: 0.1uf_0603_10V, capacitors:SMD_0603[1608], symbol capacitors_smd:0.1uf_0603_10V
Connections:
- net +5V: now also C17.1, C18.1
- net GND: now also C17.2, C18.2
Changed lines of the file:
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@@
 (kicad_sch (version 20211123) (generator eeschema)
   (paper "A4")
+  (junction (at 152.4 92.71) (diameter 0) (color 0 0 0 0)
+  )
   (junction (at 168.91 83.82) (diameter 0) (color 0 0 0 0)
   )
+  (junction (at 152.4 105.41) (diameter 0) (color 0 0 0 0)
+  )
   (junction (at 171.45 66.04) (diameter 0) (color 0 0 0 0)
   )
   (junction (at 134.62 83.82) (diameter 0) (color 0 0 0 0)
   )
+  (wire (pts (xy 152.4 105.41) (xy 157.48 105.41))
+    (stroke (width 0) (type default) (color 0 0 0 0))
+  )
   (wire (pts (xy 165.1 76.2) (xy 175.26 76.2))
     (stroke (width 0) (type default) (color 0 0 0 0))
@@
     (stroke (width 0) (type default) (color 0 0 0 0))
   )
+  (wire (pts (xy 157.48 104.14) (xy 157.48 105.41))
+    (stroke (width 0) (type default) (color 0 0 0 0))
+  )
   (wire (pts (xy 137.16 81.28) (xy 134.62 81.28))
     (stroke (width 0) (type default) (color 0 0 0 0))
   )
+  (wire (pts (xy 157.48 92.71) (xy 157.48 96.52))
+    (stroke (width 0) (type default) (color 0 0 0 0))
+  )
   (wire (pts (xy 134.62 81.28) (xy 134.62 83.82))
     (stroke (width 0) (type default) (color 0 0 0 0))
   )
+  (wire (pts (xy 147.32 92.71) (xy 152.4 92.71))
+    (stroke (width 0) (type default) (color 0 0 0 0))
+  )
   (wire (pts (xy 165.1 71.12) (xy 168.91 71.12))
     (stroke (width 0) (type default) (color 0 0 0 0))
@@
     (stroke (width 0) (type default) (color 0 0 0 0))
   )
+  (wire (pts (xy 152.4 91.44) (xy 152.4 92.71))
+    (stroke (width 0) (type default) (color 0 0 0 0))
+  )
   (wire (pts (xy 116.84 78.74) (xy 137.16 78.74))
     (stroke (width 0) (type default) (color 0 0 0 0))
   )
+  (wire (pts (xy 147.32 104.14) (xy 147.32 105.41))
+    (stroke (width 0) (type default) (color 0 0 0 0))
+  )
   (wire (pts (xy 134.62 83.82) (xy 134.62 87.63))
     (stroke (width 0) (type default) (color 0 0 0 0))
@@
     (stroke (width 0) (type default) (color 0 0 0 0))
   )
+  (wire (pts (xy 147.32 105.41) (xy 152.4 105.41))
+    (stroke (width 0) (type default) (color 0 0 0 0))
+  )
   (wire (pts (xy 165.1 81.28) (xy 175.26 81.28))
+    (stroke (width 0) (type default) (color 0 0 0 0))
+  )
+  (wire (pts (xy 147.32 92.71) (xy 147.32 96.52))
+    (stroke (width 0) (type default) (color 0 0 0 0))
+  )
+  (wire (pts (xy 152.4 92.71) (xy 157.48 92.71))
+    (stroke (width 0) (type default) (color 0 0 0 0))
+  )
+  (wire (pts (xy 152.4 105.41) (xy 152.4 106.68))
     (stroke (width 0) (type default) (color 0 0 0 0))
   )
@@
     (pin "9")
   )
+  (symbol (lib_id "power:+5V") (at 152.4 91.44 0) (unit 1)
+    (in_bom yes) (on_board yes) (fields_autoplaced)
+    (property "Reference" "#PWR017" (id 0) (at 152.4 95.25 0)
+      (effects (font (size 1.27 1.27)) hide)
+    )
+    (property "Value" "+5V" (id 1) (at 152.4 86.36 0))
+    (property "Footprint" "" (id 2) (at 152.4 91.44 0)
+      (effects (font (size 1.27 1.27)) hide)
+    )
+    (property "Datasheet" "" (id 3) (at 152.4 91.44 0)
+      (effects (font (size 1.27 1.27)) hide)
+    )
+    (pin "1")
+  )
+  (symbol (lib_id "capacitors_smd:0.1uf_0603_10V") (at 157.48 100.33 0) (unit 1)
+    (in_bom yes) (on_board yes) (fields_autoplaced)
+    (property "Reference" "C18" (id 0) (at 161.29 99.0599 0)
+      (effects (font (size 1.27 1.27)) (justify left))
+    )
+    (property "Value" "0.1uf_0603_10V" (id 1) (at 158.115 102.87 0)
+      (effects (font (size 1.27 1.27)) (justify left) hide)
+    )
+    (property "Footprint" "capacitors:SMD_0603[1608]" (id 2) (at 158.75 85.09 0)
+      (effects (font (size 1.27 1.27)) hide)
+    )
+    (property "Datasheet" "https://www.mouser.com/datasheet/2/445/885012206020-1727542.pdf" (id 3) (at 160.02 114.3 0)
+      (effects (font (size 1.27 1.27)) hide)
+    )
+    (property "Manufacturer" "Wurth Elektronik " (id 4) (at 158.75 116.84 0)
+      (effects (font (size 1.27 1.27)) hide)
+    )
+    (property "Part Number" "885012206020" (id 5) (at 157.48 87.63 0)
+      (effects (font (size 1.524 1.524)) hide)
+    )
+    (property "Display" "0u1" (id 6) (at 161.29 101.5999 0)
+      (effects (font (size 1.27 1.27)) (justify left))
+    )
+    (property "IPN" "CAP-005-0000" (id 7) (at 158.115 72.39 0)
+      (effects (font (size 1.27 1.27)) (justify left) hide)
+    )
+    (pin "1")
+    (pin "2")
+  )
   (symbol (lib_id "power:GND") (at 134.62 87.63 0) (unit 1)
     (in_bom yes) (on_board yes) (fields_autoplaced)
@@
       (effects (font (size 1.27 1.27)) hide)
     )
+    (pin "1")
+  )
+  (symbol (lib_id "capacitors_smd:10uf_0603_25V") (at 147.32 100.33 0) (unit 1)
+    (in_bom yes) (on_board yes)
+    (property "Reference" "C17" (id 0) (at 151.13 97.79 0)
+      (effects (font (size 1.27 1.27)) (justify left))
+    )
+    (property "Value" "10uf_0603_25V" (id 1) (at 147.955 102.87 0)
+      (effects (font (size 1.27 1.27)) (justify left) hide)
+    )
+    (property "Footprint" "capacitors:SMD_0603[1608]" (id 2) (at 148.59 85.09 0)
+      (effects (font (size 1.27 1.27)) hide)
+    )
+    (property "Datasheet" "https://search.murata.co.jp/Ceramy/image/img/A01X/G101/ENG/GRT188R61E106ME13-01.pdf" (id 3) (at 149.86 114.3 0)
+      (effects (font (size 1.27 1.27)) hide)
+    )
+    (property "Manufacturer" "Murata Electronics" (id 4) (at 148.59 116.84 0)
+      (effects (font (size 1.27 1.27)) hide)
+    )
+    (property "Part Number" "GRT188R61E106ME13D" (id 5) (at 147.32 87.63 0)
+      (effects (font (size 1.524 1.524)) hide)
+    )
+    (property "Display" "10u" (id 6) (at 151.13 100.33 0)
+      (effects (font (size 1.27 1.27)) (justify left))
+    )
+    (property "IPN" "CAP-011-0000" (id 7) (at 147.955 72.39 0)
+      (effects (font (size 1.27 1.27)) (justify left) hide)
+    )
+    (pin "1")
+    (pin "2")
+  )
+  (symbol (lib_id "power:GND") (at 152.4 106.68 0) (unit 1)
+    (in_bom yes) (on_board yes) (fields_autoplaced)
+    (property "Reference" "#PWR019" (id 0) (at 152.4 113.03 0)
+      (effects (font (size 1.27 1.27)) hide)
+    )
+    (property "Value" "GND" (id 1) (at 152.4 111.76 0))
+    (property "Footprint" "" (id 2) (at 152.4 106.68 0)
+      (effects (font (size 1.27 1.27)) hide)
+    )
+    (property "Datasheet" "" (id 3) (at 152.4 106.68 0)
+      (effects (font (size 1.27 1.27)) hide)
+    )
